File: Schematic and PCB/ESP32C6-dev-board.kicad_sch (KiCad schematic)
At the start: 19 parts, among them J1 Conn_01x15_Pin, J2 Conn_01x02_Pin, J3 Conn_01x02_Pin, J4 Conn_01x02_Pin, U1 Seeed Studio XIAO SAMD21, U2 AMS1117-3.3, U3 LM35-LP, U4 DHT11

Commit message: finished modifications for R01
Parts:
- removed C2: 10u, Capacitor_SMD:CP_Elec_4x5.4, symbol Device:C_Polarized
- removed C4, C5, C6: 100n, Capacitor_SMD:C_0805_2012Metric, symbol Device:C
- removed D1: WS2812, LED_SMD:LED_WS2812_PLCC6_5.0x5.0mm_P1.6mm, symbol LED:WS2812
- removed J3: Conn_01x02_Pin, Connector_PinHeader_2.54mm:PinHeader_1x02_P2.54mm_Vertical, symbol Connector:Conn_01x02_Pin
- removed R2: 10k, Resistor_SMD:R_0805_2012Metric, symbol Device:R
- removed U2: AMS1117-3.3, Package_TO_SOT_SMD:SOT-223-3_TabPin2, symbol Regulator_Linear:AMS1117-3.3
- removed U3: LM35-LP, Package_TO_SOT_THT:TO-92_Inline, symbol Sensor_Temperature:LM35-LP
- removed U4: DHT11, Sensor:Aosong_DHT11_5.5x12.0_P2.54mm, symbol Sensor:DHT11
- added D2: WS2812B, LED_SMD:LED_WS2812B_PLCC4_5.0x5.0mm_P3.2mm, symbol LED:WS2812B
- added J3: Conn_01x04_Pin, Connector_PinHeader_2.54mm:PinHeader_1x04_P2.54mm_Vertical, symbol Connector:Conn_01x04_Pin
- added J5: Conn_01x02_Pin, Connector_PinHeader_2.54mm:PinHeader_1x02_P2.54mm_Vertical, symbol Connector:Conn_01x02_Pin
- added R2: R_Photo, OptoDevice:R_LDR_5.0x4.1mm_P3mm_Vertical, symbol Device:R_Photo
- added R5: 330, Resistor_SMD:R_0805_2012Metric, symbol Device:R
- R4: value 470 -> 330
Connections:
- net 3V3: now also J5.1 (Pin_1), R2.1
- net D1-A1: now also J4.1 (Pin_1)
- net D4-SDA: now also R5.1; no longer J4.1 (Pin_1)
- net D5-SCL: now also R4.1
- net GND: now also R1.1, D2.3 (VSS), J3.2 (Pin_2)
- net VIN: now also C1.1, C3.1, D2.1 (VDD)
- net at J2.2 (Pin_2), R1.2: now also R2.2
- net at R3.1: now also D2.4 (DIN)
- net at R4.2: now also J3.3 (Pin_3)
- removed net 5V: C1.1, C3.1, J1.14 (Pin_14), R4.1
- new net: J3.1 (Pin_1), J5.2 (Pin_2)
- new net: J3.4 (Pin_4), R5.2
Other:
- moved on the sheet: R1
